File: RIAA.kicad_pcb (KiCad board)
At the start: 2 copper layers, 112 x 202 mm, 44 parts, among them K1 G6K-2, P1 Fra Hovedprint, P2 Fra Ledning, U2 LM317_TO-220, U3 OPA2134

Commit message: feat:
Parts:
- P1: value Fra Hovedprint -> From main PCB
- P2: value Fra Ledning -> From Wire
- moved C4 67.0 mm to (152.5, 143.5)
- moved C5 67.0 mm to (152.7, 154.6)
- moved C2 30.8 mm to (173.1, 142.9), turned to 180 degrees
- moved C7 22.5 mm to (186.5, 129.5)
- moved C1 20.5 mm to (182.2, 147.3)
- moved C9 5.08 mm to (183.5, 139.1), turned to 0 degrees
- moved C12 0.19 mm to (213.6, 200.0)
Connections:
- K1 pad 4: GND -> unconnected-(K1-Pad4)
- K1 pad 5: GND -> unconnected-(K1-Pad5)
Routing:
- net L OUT: track 4.35 -> 200.1 mm, vias 0 -> 1
- net R OUT: track 5.29 -> 164.7 mm, vias 0 -> 2
- net R IN PICKUP: track 5.52 -> 146.7 mm
- net L IN PICKUP: track 5.05 -> 111.4 mm
- net Net-(U3C-V-): track 0.00 -> 83.6 mm, vias 0 -> 2
- net GND: track 66.7 -> 12.1 mm
- net Net-(C16-Pad1): track 25.1 -> 63.6 mm
- net Net-(U3A--): track 3.11 -> 24.0 mm
- net Net-(C11-Pad1): track 25.2 -> 43.9 mm
- net Net-(U3A-+): track 8.94 -> 25.6 mm
- net Net-(U3B--): track 3.17 -> 19.2 mm
- net Net-(U3B-+): track 9.72 -> 23.4 mm
- net 21V: track 57.0 -> 47.4 mm
- net Net-(D2-A): track 46.1 -> 48.1 mm
- net Net-(BC1-B): track 51.8 -> 52.7 mm
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
Commit message: feat:
Parts:
- renumbered P1 to P8, P2 to P9
Routing:
- net Net-(BC1-C): track 40.0 -> 48.1 mm
- net L IN PICKUP: track 111.4 -> 113.5 mm
- net R IN PICKUP: track 146.7 -> 145.0 mm
- added copper zone on F.Cu, net GND
- removed copper zone on B.Cu, net (none)
- removed copper zone on F.Cu, net (none)
