File: RIAA.kicad_sch (KiCad schematic)
At the start: 64 parts, among them K1 G6K-2, P10 From Keyboard, P8 From main PCB, P9 From Wire, U5 OPA2134, U6 OPA2134, U7 LM317_TO-220

Commit message: WIP: Working on SMD.
Parts:
- C27, C28, C32: LSCS PN (none) -> C24497
- C29: footprint Capacitor_SMD:CP_Elec_5x5.4 -> Capacitor_SMD:C_1206_3216Metric_Pad1.33x1.80mm_HandSolder; LSCS PN (none) -> C24497
- C30: footprint Capacitor_SMD:CP_Elec_5x5.4 -> Capacitor_SMD:C_1206_3216Metric_Pad1.33x1.80mm_HandSolder; LSCS PN (none) -> C13585
- C33: LSCS PN (none) -> C7432784
- D5: footprint Diode_SMD:D_MiniMELF -> Diode_SMD:D_SMA; LSCS PN (none) -> C433394
- D6: footprint Diode_SMD:D_MiniMELF -> Diode_SMD:D_SMA; LSCS PN (none) -> C433393
- K1: LSCS PN (none) -> C5278023
- R19: LSCS PN (none) -> C870816
- R20: LSCS PN (none) -> C870638
- R21: LSCS PN (none) -> C4410
- R22: LSCS PN (none) -> C17900
- U5, U6: LSCS PN (none) -> C87361
- U7: footprint Package_TO_SOT_SMD:TO-252-3_TabPin2 -> Package_TO_SOT_SMD:TO-263-3_TabPin2; LSCS PN (none) -> C88007
Changed lines of the file:
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@@
 			)
 		)
-		(property "Datasheet" "http://omronfs.omron.com/en_US/ecb/products/pdf/en-g6k.pdf"
+		(property "Datasheet" "http://omronfs.omron.com/en_US/ecb/products/pdf/en-g6k.pdf, https://jlcpcb.com/partdetail/OmronElectronics-G6K_2F_Y_TRDC24/C5278023"
 			(at 270.51 185.42 0)
 			(effects
@@
 			)
 		)
-		(property "Description" "Miniature 2-pole relay, Single-side Stable"
+		(property "Description" "Miniature 2-pole relay, Single-side Stable, 24V"
 			(at 270.51 185.42 0)
 			(effects
@@
 			)
 		)
+		(property "LSCS PN" "C5278023"
+			(at 270.51 185.42 0)
+			(effects
+				(font
+					(size 1.27 1.27)
+				)
+			)
+		)
 		(pin "8"
 		)
@@
 			)
 		)
-		(property "Datasheet" "~"
+		(property "Datasheet" "https://jlcpcb.com/partdetail/YAGEO-RT1206BRD075K6L/C870816"
 			(at 77.47 175.26 0)
 			(effects
@@
 			)
 		)
+		(property "LSCS PN" "C870816"
+			(at 77.47 175.26 0)
+			(effects
+				(font
+					(size 1.27 1.27)
+				)
+			)
+		)
 		(pin "2"
 		)
@@
 			)
 		)
-		(property "Footprint" "Package_TO_SOT_SMD:TO-252-3_TabPin2"
+		(property "Footprint" "Package_TO_SOT_SMD:TO-263-3_TabPin2"
 			(at 77.47 153.67 0)
 			(effects
@@
 					(italic yes)
 				)
+				(hide yes)
 			)
 		)
-		(property "Datasheet" "http://www.ti.com/lit/ds/symlink/lm317.pdf"
+		(property "Datasheet" "http://www.ti.com/lit/ds/symlink/lm317.pdf, https://jlcpcb.com/partdetail/TexasInstruments-LM317KTTR/C88007"
 			(at 77.47 160.02 0)
 			(effects
@@
 			)
 		)
+		(property "LSCS PN" "C88007"
+			(at 77.47 160.02 0)
+			(effects
+				(font
+					(size 1.27 1.27)
+				)
+			)
+		)
 		(pin "3"
 		)
@@
 			)
 		)
-		(property "Datasheet" "http://www.ti.com/lit/ds/symlink/opa134.pdf"
+		(property "Datasheet" "http://www.ti.com/lit/ds/symlink/opa134.pdf,https://jlcpcb.com/partdetail/TexasInstruments-OPA2134UA2K5/C87361"
 			(at 303.53 82.55 0)
 			(effects
@@
 			)
 		)
+		(property "LSCS PN" "C87361"
+			(at 303.53 82.55 0)
+			(effects
+				(font
+					(size 1.27 1.27)
+				)
+			)
+		)
 		(pin "8"
 		)
@@
 			)
 		)
-		(property "Datasheet" "~"
+		(property "Datasheet" "https://jlcpcb.com/partdetail/YAGEO-RT1206BRD07300RL/C870638"
 			(at 93.98 165.1 0)
 			(effects
@@
 			)
 		)
+		(property "LSCS PN" "C870638"
+			(at 93.98 165.1 0)
+			(effects
+				(font
+					(size 1.27 1.27)
+				)
+			)
+		)
 		(pin "2"
 		)
@@
 			)
 		)
+		(property "LSCS PN" "C24497"
+			(at 25.4 81.28 90)
+			(effects
+				(font
+					(size 1.27 1.27)
+				)
+			)
+		)
 		(pin "1"
 		)
@@
 			)
 		)
-		(property "Datasheet" "~"
+		(property "Datasheet" "https://jlcpcb.com/partdetail/4817-1206W4F1001T5E/C4410"
 			(at 243.84 138.43 0)
 			(effects
@@
 			)
 		)
+		(property "LSCS PN" "C4410"
+			(at 243.84 138.43 90)
+			(effects
+				(font
+					(size 1.27 1.27)
+				)
+			)
+		)
 		(pin "2"
 		)
@@
 			)
 		)
-		(property "Datasheet" "~"
+		(property "Datasheet" "https://jlcpcb.com/partdetail/18588-1206W4F1003T5E/C17900"
 			(at 243.84 158.75 0)
 			(effects
@@
 			)
 		)
+		(property "LSCS PN" "C17900"
+			(at 243.84 158.75 90)
+			(effects
+				(font
+					(size 1.27 1.27)
+				)
+			)
+		)
 		(pin "2"
 		)
@@
 			)
 		)
-		(property "Datasheet" "http://www.ti.com/lit/ds/symlink/opa134.pdf"
+		(property "Datasheet" "http://www.ti.com/lit/ds/symlink/opa134.pdf,https://jlcpcb.com/partdetail/TexasInstruments-OPA2134UA2K5/C87361"
 			(at 40.64 93.98 0)
 			(effects
@@
 			)
 		)
+		(property "LSCS PN" "C87361"
+			(at 40.64 93.98 0)
+			(effects
+				(font
+					(size 1.27 1.27)
+				)
+				(hide yes)
+			)
+		)
 		(pin "8"
 		)
@@
 			)
 		)
-		(property "Datasheet" "http://www.ti.com/lit/ds/symlink/opa134.pdf"
+		(property "Datasheet" "http://www.ti.com/lit/ds/symlink/opa134.pdf,https://jlcpcb.com/partdetail/TexasInstruments-OPA2134UA2K5/C87361"
 			(at 24.13 93.98 0)
 			(effects
@@
 			)
 		)
+		(property "LSCS PN" "C87361"
+			(at 24.13 93.98 0)
+			(effects
+				(font
+					(size 1.27 1.27)
+				)
+				(hide yes)
+			)
+		)
 		(pin "8"
 		)
@@
 			)
 		)
-		(property "Datasheet" "http://www.ti.com/lit/ds/symlink/opa134.pdf"
+		(property "Datasheet" "http://www.ti.com/lit/ds/symlink/opa134.pdf,https://jlcpcb.com/partdetail/TexasInstruments-OPA2134UA2K5/C87361"
 			(at 383.54 85.09 0)
 			(effects
@@
 			)
 		)
+		(property "LSCS PN" "C87361"
+			(at 383.54 85.09 0)
+			(effects
+				(font
+					(size 1.27 1.27)
+				)
+			)
+		)
 		(pin "8"
 		)
@@
 			)
 		)
-		(property "Footprint" "Diode_SMD:D_MiniMELF"
+		(property "Footprint" "Diode_SMD:D_SMA"
 			(at 104.14 165.1 0)
 			(effects
@@
 			)
 		)
-		(property "Datasheet" "~"
+		(property "Datasheet" "https://jlcpcb.com/partdetail/Shikues-1N4002G/C433393"
 			(at 104.14 165.1 0)
 			(effects
@@
 			)
 		)
+		(property "LSCS PN" "C433393"
+			(at 104.14 165.1 90)
+			(effects
+				(font
+					(size 1.27 1.27)
+				)
+			)
+		)
 		(pin "2"
 		)
@@
 			)
 		)
-		(property "Footprint" "Capacitor_SMD:CP_Elec_5x5.4"
+		(property "Footprint" "Capacitor_SMD:C_1206_3216Metric_Pad1.33x1.80mm_HandSolder"
 			(at 64.77 170.18 0)
 			(effects
@@
 			)
 		)
-		(property "Datasheet" "~"
+		(property "Datasheet" "https://jlcpcb.com/partdetail/25237-CL31B104KBCNNNC/C24497"
 			(at 64.77 170.18 0)
 			(effects
@@
 			)
 		)
+		(property "LSCS PN" "C24497"
+			(at 64.77 170.18 0)
+			(effects
+				(font
+					(size 1.27 1.27)
+				)
+			)
+		)
 		(pin "2"
 		)
@@
 			)
 		)
-		(property "Footprint" "Capacitor_SMD:CP_Elec_5x5.4"
+		(property "Footprint" "Capacitor_SMD:C_1206_3216Metric_Pad1.33x1.80mm_HandSolder"
 			(at 93.98 175.26 0)
 			(effects
@@
 			)
 		)
-		(property "Datasheet" "~"
+		(property "Datasheet" "https://jlcpcb.com/partdetail/14236-CL31A106KBHNNNE/C13585"
 			(at 93.98 175.26 0)
 			(effects
@@
 			)
 		)
+		(property "LSCS PN" "C13585"
+			(at 93.98 175.26 0)
+			(effects
+				(font
+					(size 1.27 1.27)
+				)
+			)
+		)
 		(pin "2"
 		)
@@
 			)
 		)
-		(property "Footprint" "Diode_SMD:D_MiniMELF"
+		(property "Footprint" "Diode_SMD:D_SMA"
 			(at 78.74 148.59 0)
 			(effects
@@
 			)
 		)
-		(property "Datasheet" "~"
+		(property "Datasheet" "https://jlcpcb.com/partdetail/Shikues-1N4004G/C433394"
 			(at 78.74 148.59 0)
 			(effects
@@
 			)
 		)
+		(property "LSCS PN" "C433394"
+			(at 78.74 148.59 0)
+			(effects
+				(font
+					(size 1.27 1.27)
+				)
+			)
+		)
 		(pin "2"
 		)
@@
 			)
 		)
-		(property "Datasheet" "http://www.ti.com/lit/ds/symlink/opa134.pdf"
+		(property "Datasheet" "http://www.ti.com/lit/ds/symlink/opa134.pdf,https://jlcpcb.com/partdetail/TexasInstruments-OPA2134UA2K5/C87361"
 			(at 115.57 82.55 0)
 			(effects
@@
 			)
 		)
+		(property "LSCS PN" "C87361"
+			(at 115.57 82.55 0)
+			(effects
+				(font
+					(size 1.27 1.27)
+				)
+			)
+		)
 		(pin "8"
 		)
@@
 			)
 		)
+		(property "LSCS PN" "C24497"
+			(at 41.91 81.28 90)
+			(effects
+				(font
+					(size 1.27 1.27)
+				)
+			)
+		)
 		(pin "1"
 		)
@@
 			)
 		)
-		(property "Datasheet" "http://www.ti.com/lit/ds/symlink/opa134.pdf"
+		(property "Datasheet" "http://www.ti.com/lit/ds/symlink/opa134.pdf,https://jlcpcb.com/partdetail/TexasInstruments-OPA2134UA2K5/C87361"
 			(at 201.93 85.09 0)
 			(effects
@@
 			)
 		)
+		(property "LSCS PN" "C87361"
+			(at 201.93 85.09 0)
+			(effects
+				(font
+					(size 1.27 1.27)
+				)
+			)
+		)
 		(pin "8"
 		)
@@
 			)
 		)
-		(property "Datasheet" "~"
+		(property "Datasheet" "https://jlcpcb.com/partdetail/Chinocera-HGC1206R5107M100NSPJ/C7432784"
 			(at 256.54 138.43 0)
 			(effects
@@
 			)
 		)
+		(property "LSCS PN" "C7432784"
+			(at 256.54 138.43 90)
+			(effects
+				(font
+					(size 1.27 1.27)
+				)
+			)
+		)
 		(pin "2"
 		)
@@
 					(size 1.27 1.27)
 				)
-				(hide yes)
 			)
 		)
@@
 			)
 		)
-		(property "Datasheet" "https://ngspice.sourceforge.io/docs/ngspice-html-manual/manual.xhtml#cha_BJTs"
+		(property "Datasheet" ""
 			(at 224.79 88.9 0)
 			(effects
@@
 			)
 		)
-		(property "Description" "Bipolar transistor symbol for simulation only, substrate tied to the emitter"
+		(property "Description" ""
 			(at 224.79 152.4 0)
 			(effects
@@
 			)
 		)
-		(property "Datasheet" "~"
+		(property "Datasheet" "https://jlcpcb.com/partdetail/25237-CL31B104KBCNNNC/C24497"
 			(at 129.54 171.45 0)
 			(effects
@@
 			)
 		)
+		(property "LSCS PN" "C24497"
+			(at 129.54 171.45 0)
+			(effects
+				(font
+					(size 1.27 1.27)
+				)
+			)
+		)

Commit message: WIP: Adding LSCS PNs.
Parts:
- added C1, C2, C3: 470uF, Capacitor_SMD:CP_Elec_10x10.5, symbol Device:C_Polarized_Small
- C106, C107, C108, C206, C207, C208: LSCS PN (none) -> C5260729
- C31: value 2200uF -> 470uF; footprint Capacitor_SMD:CP_Elec_8x6.9 -> Capacitor_SMD:CP_Elec_10x10.5; LSCS PN (none) -> C134838
- D7, D8: value 1N914 -> 1N4004; footprint Diode_SMD:D_MiniMELF -> Diode_SMD:D_SMA; LSCS PN (none) -> C433394
- R102, R103, R111, R112, R202, R203, R211, R212: LSCS PN (none) -> C351465
- R104, R204: LSCS PN (none) -> C2984516
- R105, R205: LSCS PN (none) -> C870898
- R106, R206: LSCS PN (none) -> C2092472
- R107: LSCS PN (none) -> C870623
- R108, R208: LSCS PN (none) -> C870792
- R109, R209: LSCS PN (none) -> C870770
- R110, R210: LSCS PN (none) -> C706409
- R207: LSCS PN (none) -> C870623; LSCSL PN C137334 -> (none)
- renumbered BC1 to BC548
Connections:
- net 24VDC+: now also C1.1, C2.1, C3.1
- net GND: now also C1.2, C2.2, C3.2
Other:
- moved on the sheet: C31, C32
