File: RIAA.kicad_sch (KiCad schematic)
At the start: 67 parts, among them K1 G6K-2, P10 From Keyboard, P8 From main PCB, P9 From Wire, U5 OPA2134, U6 OPA2134, U7 LM317_TO-220

Commit message: WIP: Finishing up SMD version.
Parts:
- removed BC548: NPN, Package_TO_SOT_SMD:SOT-23_Handsoldering, symbol Simulation_SPICE:NPN
- added Q1: Q_NPN_BCE, Package_TO_SOT_SMD:SOT-89-3_Handsoldering, symbol Transistor_BJT:Q_NPN_BCE
- C1, C2, C3, C31: LCSC PN (none) -> C134524; LSCS PN C134838 -> (none)
- C101, C102, C103, C104, C105, C201, C202, C203, C204, C205, P10, P8, P9, RV1, TP1, TP2: now left out of the parts list
- C106, C107, C108, C206, C207, C208: LCSC PN (none) -> C5260729; LSCS PN C5260729 -> (none)
- C27, C28, C32: LCSC PN (none) -> C24497; LSCS PN C24497 -> (none)
- C29: value 0.1uF -> 100nF; LCSC PN (none) -> C24497; LSCS PN C24497 -> (none)
- C30: LCSC PN (none) -> C13585; LSCS PN C13585 -> (none)
- C33: LCSC PN (none) -> C7432784; LSCS PN C7432784 -> (none)
- D5, D7, D8: LCSC PN (none) -> C433394; LSCS PN C433394 -> (none)
- D6: LCSC PN (none) -> C433393; LSCS PN C433393 -> (none)
- R102, R103, R111, R112, R202, R203, R211, R212: LCSC PN (none) -> C351465; LSCS PN C351465 -> (none)
- R104, R204: LCSC PN (none) -> C2984516; LSCS PN C2984516 -> (none)
- R105, R205: LCSC PN (none) -> C870898; LSCS PN C870898 -> (none)
- R106, R206: LCSC PN (none) -> C2092472; LSCS PN C2092472 -> (none)
- R107, R207: LCSC PN (none) -> C870623; LSCS PN C870623 -> (none)
- R108, R208: LCSC PN (none) -> C870792; LSCS PN C870792 -> (none)
- R109, R209: LCSC PN (none) -> C870770; LSCS PN C870770 -> (none)
- R110, R210: LCSC PN (none) -> C706409; LSCS PN C706409 -> (none)
- R19: LCSC PN (none) -> C870816; LSCS PN C870816 -> (none)
- R20: LCSC PN (none) -> C870638; LSCS PN C870638 -> (none)
- R21: LCSC PN (none) -> C4410; LSCS PN C4410 -> (none)
- R22: LCSC PN (none) -> C17900; LSCS PN C17900 -> (none)
- U5, U6: LCSC PN (none) -> C87361; LSCS PN C87361 -> (none)
- U7: LCSC PN (none) -> C88007; LSCS PN C88007 -> (none)
Connections:
- net GND: now also Q1.3 (E)
- net at D7.2 (A), K1.8: now also Q1.2 (C)
- net at C33.1, D8.2 (A), RV1.2: now also Q1.1 (B)

Commit message: WIP: Finishing up SMD version.
Parts:
- removed P10: From Keyboard, Connector_PinSocket_2.54mm:PinSocket_1x09_P2.54mm_Horizontal, symbol Connector_Generic:Conn_01x09
- removed TP1: GND TestPoint, TestPoint:TestPoint_Loop_D2.50mm_Drill1.0mm_LowProfile, symbol Connector:TestPoint
- removed TP2: 24V TP, TestPoint:TestPoint_Loop_D2.50mm_Drill1.0mm_LowProfile, symbol Connector:TestPoint
- added P10: From Keyboard, Connector_PinSocket_2.54mm:PinSocket_2x09_P2.54mm_Horizontal, symbol Connector_Generic:Conn_02x09_Odd_Even
- C101, C201: PN (none) -> WIMA FKP2
- C102: PN (none) -> KEMET MMK
- C103, C203: footprint Capacitor_THT:C_Rect_L7.2mm_W4.5mm_P5.00mm_FKS2_FKP2_MKS2_MKP2 -> Capacitor_SMD:CP_Elec_6.3x7.7; LCSC PN (none) -> C7471881
- C105, C205: PN (none) -> WIMA MKS2
- C202:  PN (none) -> KEMET MMK
- P9: LCSC PN (none) -> C40877; now in the parts list
- RV1: footprint Potentiometer_SMD:Potentiometer_Bourns_3314J_Vertical -> Potentiometer_SMD:Potentiometer_Bourns_3314G_Vertical; LSCS PN C6083402 -> C780218; now in the parts list
- U7: footprint Package_TO_SOT_SMD:TO-263-3_TabPin2 -> Package_TO_SOT_SMD:TO-263-2; LCSC PN C88007 -> C12848
Connections:
- net 21V: now also P10.11 (Pin_11), P10.12 (Pin_12)
- net 30V: now also P10.3 (Pin_3), P10.4 (Pin_4)
- net GND: now also P10.13 (Pin_13), P10.14 (Pin_14)

Commit message: WIP: Finishing up SMD version.
Parts:
- removed P8: From main PCB, Connector_PinSocket_2.54mm:PinSocket_1x09_P2.54mm_Horizontal, symbol Connector_Generic:Conn_01x09
- added P8: From main PCB, Connector_PinSocket_2.54mm:PinSocket_2x09_P2.54mm_Horizontal, symbol Connector_Generic:Conn_02x09_Odd_Even
Connections:
- net 21V: now also P8.15 (Pin_15), P8.16 (Pin_16)
- net 30V: now also P8.17 (Pin_17), P8.18 (Pin_18)
- net GND: now also P8.10 (Pin_10), P8.13 (Pin_13), P8.14 (Pin_14), P8.3 (Pin_3), P8.4 (Pin_4), P8.5 (Pin_5), P8.6 (Pin_6), P8.9 (Pin_9)
- net L IN PICKUP: now also P8.7 (Pin_7), P8.8 (Pin_8)
- net R IN PICKUP: now also P8.11 (Pin_11), P8.12 (Pin_12)
- net RELAY ON: now also P8.1 (Pin_1), P8.2 (Pin_2)
