File: RIAA.kicad_sch (KiCad schematic)
At the start: 65 parts, among them K1 G6K-2, P10 From Keyboard, P8 From main PCB, P9 From Wire, Q1 Q_NPN_BCE, U5 OPA2134, U6 OPA2134, U7 LM317_TO-220

Commit message: Set up repository for open-source community development
- Relicense: CERN-OHL-S v2 for hardware, CC BY-SA 4.0 for docs,
  GPL-3.0-or-later for scripts.
- Stop tracking generated and per-user files (production zips, backups,
  v1 gerbers, .kicad_prl, .wbk); extend .gitignore accordingly.
- Remove unused 3314J trimmer library.
- Fix misspelled "LSCS PN" / " PN" fields so K1 and RV1 appear in the BOM.
- Add KiCad CI: DRC (blocking), ERC (report-only), schematic PDF, gerbers,
  full + JLCPCB BOM/CPL, renders, and draft releases on v* tags.
- Add scripts/make_bom.py to include hand-soldered parts in the full BOM.
- Rewrite README (pinouts, build steps, known issues), add design notes,
  CONTRIBUTING, CHANGELOG, issue and PR templates.

Co-Authored-By: Claude Opus 5.5 <noreply@anthropic.com>
Parts:
- C202:  PN KEMET MMK -> (none); PN (none) -> KEMET MMK
- K1: LCSC PN (none) -> C5278023; LSCS PN C5278023 -> (none)
- RV1: LCSC PN (none) -> C780218; LSCS PN C780218 -> (none)
Changed lines of the file:
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@@
 			)
 		)
-		(property "LSCS PN" "C5278023"
+		(property "LCSC PN" "C5278023"
 			(at 270.51 185.42 0)
 			(effects
@@
 			)
 		)
-		(property "LSCS PN" "C780218"
+		(property "LCSC PN" "C780218"
 			(at 262.89 158.75 90)
 			(effects
@@
 			)
 		)
-		(property " PN" "KEMET MMK"
+		(property "PN" "KEMET MMK"
 			(at 298.45 97.79 90)
 			(effects
