File: RIAA.kicad_sch (KiCad schematic)
At the start: 65 parts, among them K1 G6K-2, P10 From Keyboard, P8 From main PCB, P9 From Wire, Q1 Q_NPN_BCE, U5 OPA2134, U6 OPA2134, U7 LM317_TO-220

Commit message: Added RIAA response and optimized layout.
Parts:
- removed C104, C204: 2uF, Capacitor_THT:C_Rect_L7.2mm_W4.5mm_P5.00mm_FKS2_FKP2_MKS2_MKP2, symbol Device:C
- removed C2, C3, C31: 470uF, Capacitor_SMD:CP_Elec_10x10.5, symbol Device:C_Polarized_Small
- removed C32: 100nF, Capacitor_SMD:C_1206_3216Metric_Pad1.33x1.80mm_HandSolder, symbol Device:C
- removed R102, R111, R112, R202, R211, R212: 47k, Resistor_SMD:R_1206_3216Metric_Pad1.30x1.75mm_HandSolder, symbol Device:R
- added C34, C35: 10uF, Capacitor_SMD:CP_Elec_5x5.4, symbol Device:C_Polarized_Small
- added NT1, NT2: NetTie_2, NetTie:NetTie-2_SMD_Pad0.5mm, symbol Device:NetTie_2
- added R23, R24, R25, R26: 100k, Resistor_SMD:R_1206_3216Metric_Pad1.30x1.75mm_HandSolder, symbol Device:R
- C102, C202: value 39nF -> 33nF; PN KEMET MMK -> WIMA MKS2
- C103, C203: value 200uF -> 220uF; now in the parts list
- Q1: value Q_NPN_BCE -> BCV49; LCSC PN C21714170 -> C526472
- R104, R204: value 499 -> 590; LCSC PN C2984516 -> C870807
- R105, R205: value 80.6k -> 95.3k; LCSC PN C870898 -> C274048
- R106, R206: value 8.45k -> 10k; LCSC PN C2092472 -> C136889
- R108, R208: LCSC PN C870792 -> C488896
- R19: value 5k6 -> 4k7; LCSC PN C870816 -> C17936
Connections:
- net 24VDC+: now also R23.1, R25.1; no longer R103.1, R203.1
- net GND: now also C34.2, C35.2, NT1.2, NT2.2, R24.2, R26.2; no longer P8.10 (Pin_10), P8.13 (Pin_13), P8.14 (Pin_14), P8.9 (Pin_9)
- net at R107.1, R108.1: now also C105.2, U5.5 (+)
- net at C205.2, U6.5 (+): now also R207.1, R208.1
- new net GND L IN PICKUP: NT1.1, P8.10 (Pin_10), P8.9 (Pin_9)
- new net GND R IN PICKUP: NT2.1, P8.13 (Pin_13), P8.14 (Pin_14)
- new net VREF_L: C34.1, R103.1, R23.2, R24.1
- new net VREF_R: C35.1, R203.1, R25.2, R26.1
- no-connect marks 0 -> 15
Other:
- note added: "NT1: star point. The L pickup return (P8 9/10) joins GND only here, at the C101 GND pad."
- note added: "NT2: star point. The R pickup return (P8 13/14) joins GND only here, at the C201 GND pad."
- note added: "Q1 must be a Darlington (BCV49), like 8IC1 (MPSA13) on the original B&O board. A single NPN gets too little base current via R22+RV1 at long delays: late or no pull-in."
- note added: "Relay notes: 8RL1 on the original B&O PCB 8, B&O pin numbers (orig. P8 pin n = P8 pins 2n-1/2n here) - G6K P1 to D2 cathode - G6K P2 to P8-6 (R OUT RIAA) & P9-3 (R OUT) - G6K P3 to P9-5 (GND) - G6K P4 to P9-5 (GND) - G6K P5 to P9-5 (GND) - G6K P6 to P9-5 (GND) - G6K P7 to P8-4 (L OUT RIAA) & P9-1 (L OUT) - G6K P8 to D2 anode"
- note added: "VREF = 24VDC+ / 2, filtered (100k || 100k, 10 uF). Rail ripple reaches the output at -42 dB (100 Hz) instead of +13 dB with a plain 47k/47k divider. Feeds the stage 1 + inputs via R103/R203 (47k = cartridge load). Stage 2 is DC-coupled to stage 1."
- note removed: "Relay Notes - G6K P1 to D2 cathode - G6K P2 to P8-6 (R OUT RIAA) & P9-3 (R OUT) - G6K P3 to P9-5 (GND) - G6K P4 to P9-5 (GND) - G6K P5 to P9-5 (GND) - G6K P6 to P9-5 (GND) - G6K P7 to P8-4 (L OUT RIAA) & P9-1 (L OUT) - G6K P8 to D2 anode"
